File: hardware/boards/teensy-eurorack.kicad_pcb (KiCad board)
At the start: 4 copper layers, 64.8 x 109.2 mm, 51 parts, among them J27 Conn_01x02, J28 Conn_02x08_Odd_Even, U2 AD5754BREZ, U3 AD5754BREZ, U4 Teensy4.1, U5 MCP1700-2502E, U6 AD7606BSTZ, U7 6N138

Commit message: pull changes from schematic, reroute as double layer board
Parts:
- removed REF**: teensy-eurorack-lite-breakout, footprints:teensy-eurorack-lite-breakout
- moved J27 5.68 mm to (121.9, 48.3), turned to 0 degrees
Connections:
- R1 pad 2: Net-(R1-Pad2) -> /ADC_RESET
- R2 pad 1: Net-(R2-Pad1) -> +3V3
- R2 pad 2: GND -> Net-(R2-Pad2)
- U4 pad 16: Net-(U4-Pad16) -> /IN2
- U4 pad 17: Net-(U4-Pad17) -> /IN1
- U4 pad 20: Net-(U4-Pad20) -> /ENC1A
- U4 pad 21: Net-(U4-Pad21) -> /ENC1B
- U4 pad 22: Net-(U4-Pad22) -> /ENC1SW
- U4 pad 30: /IN1 -> Net-(U4-Pad30)
- U4 pad 31: /IN2 -> Net-(U4-Pad31)
- U4 pad 6: Net-(U4-Pad6) -> /ADC_RESET
- U6 pad 11: Net-(R1-Pad2) -> /ADC_RESET
- U6 pad 8: Net-(R2-Pad1) -> Net-(R2-Pad2)
Routing:
- net /ADC_RESET: track 0.00 -> 58.9 mm, vias 0 -> 1
- net +5V: track 211.7 -> 187.4 mm
- net /ADC_CS: track 76.2 -> 99.8 mm, vias 2 -> 1
- net /ENC1A: track 0.00 -> 21.7 mm
- net /ENC1B: track 0.00 -> 18.1 mm
- net -12V: track 95.7 -> 110.5 mm, vias 2 -> 0
- net /ENC1SW: track 0.00 -> 14.5 mm
- net /IN1: track 56.7 -> 43.6 mm, vias 2 -> 1
- net Net-(R1-Pad2): track 10.7 -> 0.00 mm
- net /IN2: track 53.9 -> 43.6 mm, vias 1 -> 0
- net /DAC_SYNC: track 79.4 -> 87.2 mm
- net /ADC_SCK: track 75.3 -> 83.1 mm, vias 2 -> 1
- net Net-(R2-Pad2): track 0.00 -> 7.66 mm
- net /VOUT8: track 18.9 -> 24.8 mm, vias 1 -> 2
- net GND: track 55.2 -> 49.5 mm, vias 46 -> 50
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- added copper zone on B.Cu, net GND
Other:
- copper layers 4 -> 2
- board text added: "ADC_RESET"
- board text added: "Teensy eurorack control voltage shield v0.2"
- board text removed: "Teensy eurorack lite shield v0.1"

Commit message: rerouted pcb
Parts:
- removed R2: 4.7k, Resistor_SMD:R_0805_2012Metric
- added J1: Conn_01x03, Pin_Headers:Pin_Header_Straight_1x03_Pitch2.54mm, B.Cu at (153.0, 115.6)
- added J2: Conn_01x02, Pin_Headers:Pin_Header_Straight_1x02_Pitch2.54mm, B.Cu at (161.9, 114.8)
- added J3: Conn_01x03, Pin_Headers:Pin_Header_Straight_1x03_Pitch2.54mm, B.Cu at (153.0, 111.8)
- C19, C21, C23, C25, C31, C32, C33, C34: footprint Capacitor_SMD:C_0805_2012Metric -> Capacitors_THT:CP_Radial_D5.0mm_P2.00mm
- moved C19 29.0 mm to (143.5, 50.8)
- moved C33 27.9 mm to (166.4, 50.8)
- moved C39 17.0 mm to (149.1, 87.9)
- moved C34 15.9 mm to (158.8, 50.8)
- moved C29 14.4 mm to (145.4, 87.9)
- moved C21 14.0 mm to (151.1, 50.8)
- moved C37 12.2 mm to (145.4, 66.0)
- moved C30 9.52 mm to (149.2, 66.0)
- moved C25 8.52 mm to (151.1, 57.1)
- moved C31 8.52 mm to (158.8, 57.1)
- moved C27 6.20 mm to (141.6, 80.1)
- moved U2 5.89 mm to (156.7, 66.0)
- moved U5 5.24 mm to (143.5, 73.0)
- moved C20 5.08 mm to (166.4, 91.4)
- moved C24 5.08 mm to (166.4, 87.6)
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Connections:
- BB1 pad 20: Net-(BB1-Pad20) -> (no net)
- BB1 pad 41: Net-(BB1-Pad41) -> (no net)
- BB1 pad 42: Net-(BB1-Pad42) -> (no net)
- BB1 pad 43: Net-(BB1-Pad43) -> (no net)
- BB1 pad 53: Net-(BB1-Pad53) -> (no net)
- BB1 pad 54: Net-(BB1-Pad54) -> (no net)
- BB1 pad 55: Net-(BB1-Pad55) -> (no net)
- BB1 pad 56: Net-(BB1-Pad56) -> (no net)
- J28 pad 13: Net-(J28-Pad13) -> (no net)
- J28 pad 14: Net-(J28-Pad14) -> (no net)
- J28 pad 15: Net-(J28-Pad15) -> (no net)
- J28 pad 16: Net-(J28-Pad16) -> (no net)
- U2 pad 12: Net-(U2-Pad12) -> (no net)
- U2 pad 13: Net-(U2-Pad13) -> (no net)
- U2 pad 2: Net-(U2-Pad2) -> (no net)
- U2 pad 6: Net-(U2-Pad6) -> (no net)
- U3 pad 12: Net-(U3-Pad12) -> (no net)
- U3 pad 13: Net-(U3-Pad13) -> (no net)
- U3 pad 16: /DAC_SDOUT -> (no net)
- U3 pad 2: Net-(U3-Pad2) -> (no net)
- U3 pad 6: Net-(U3-Pad6) -> (no net)
- U4 pad 10: Net-(U4-Pad10) -> (no net)
- U4 pad 11: Net-(U4-Pad11) -> (no net)
- U4 pad 12: Net-(U4-Pad12) -> (no net)
- U4 pad 14: Net-(U4-Pad14) -> (no net)
- U4 pad 15: Net-(U4-Pad15) -> (no net)
- U4 pad 23: /DAC_SCK -> (no net)
- U4 pad 24: Net-(U4-Pad24) -> (no net)
- U4 pad 25: Net-(U4-Pad25) -> (no net)
- U4 pad 26: /ADC_MISO -> (no net)
- U4 pad 27: Net-(U4-Pad27) -> (no net)
- U4 pad 29: /ADC_SCK -> /ADC_RANGE
- U4 pad 30: Net-(U4-Pad30) -> /DAC_SYNC
- U4 pad 31: Net-(U4-Pad31) -> (no net)
- U4 pad 32: Net-(U4-Pad32) -> (no net)
- U4 pad 33: /DAC_SDOUT -> /MISO1
- U4 pad 36: Net-(U4-Pad36) -> (no net)
- U4 pad 37: Net-(U4-Pad37) -> (no net)
- U4 pad 38: /DAC_SYNC -> (no net)
- U4 pad 39: Net-(U4-Pad39) -> (no net)
- U4 pad 40: Net-(U4-Pad40) -> (no net)
- U4 pad 41: Net-(U4-Pad41) -> (no net)
- U4 pad 42: Net-(U4-Pad42) -> (no net)
- U4 pad 43: Net-(U4-Pad43) -> (no net)
- U4 pad 44: Net-(U4-Pad44) -> (no net)
- U4 pad 45: Net-(U4-Pad45) -> (no net)
- U4 pad 9: Net-(U4-Pad9) -> (no net)
- U6 pad 15: Net-(U6-Pad15) -> (no net)
- U6 pad 42: Net-(U6-Pad42) -> (no net)
- U6 pad 8: Net-(R2-Pad2) -> /ADC_RANGE
- U7 pad 1: Net-(U7-Pad1) -> (no net)
- U7 pad 4: Net-(U7-Pad4) -> (no net)
- U7 pad 7: Net-(U7-Pad7) -> (no net)
Routing:
- net /ADC_RANGE: track 0.00 -> 86.9 mm, vias 0 -> 1
- net /DAC_SDOUT: track 55.6 -> 0.00 mm, vias 1 -> 0
- net +5V: track 187.4 -> 230.1 mm, vias 3 -> 2
- net /ADC_MISO: track 72.0 -> 42.2 mm
- net GND: track 49.5 -> 77.2 mm, vias 50 -> 464
- net /MISO1: track 0.00 -> 27.7 mm
- net /ADC_SCK: track 83.1 -> 56.9 mm, vias 1 -> 2
- net /ADC_CS: track 99.8 -> 80.3 mm, vias 1 -> 2
- net +3V3: track 189.0 -> 208.5 mm, vias 4 -> 0
- net /VOUT8: track 24.8 -> 43.5 mm, vias 2 -> 0
- net /VGND8: track 62.4 -> 80.0 mm
- net Net-(U2-Pad16): track 21.9 -> 35.2 mm
- net /IN1: track 43.6 -> 54.1 mm, vias 1 -> 0
- net /DAC_SYNC: track 87.2 -> 76.8 mm, vias 3 -> 2
- net /TFT_SCK: track 68.4 -> 58.5 mm
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Other:
- board text added: "J1, J3: Select SPI1 for ADC to use SPI1 (share with DAC) Select SPI2 for ADC to use SPI2 (share with flash)"
- board text added: "J2: if you are using SPI2 for ADC: connect MISO2 to pin 54 connect SCK2 to pin 49 (on underneath teensy 4.1)"
- board text added: "PIN 1"
- board text added: "SPI1"
- board text added: "SPI2"
- board text added: "eurorack control voltage v0.3"
- board text added: "https://github.com/newdigate/teensy-control-voltage version 0.3"
- board text removed: "Teensy 4.1"
- board text removed: "Teensy eurorack control voltage shield v0.2"
- board text removed: "https://github.com/newdigate version 0.1"
