File: hardware/boards/teensy-eurorack.sch (KiCad schematic (older format))
At the start: 50 parts, among them J27 Conn_01x02, J28 Conn_02x08_Odd_Even, U2 AD5754BREZ, U3 AD5754BREZ, U4 Teensy4.1, U5 MCP1700-2502E, U6 AD7606BSTZ, U7 6N138

Commit message: updated schematic with jumpers to configure ADC to use either SPI1 or SPI2
Parts:
- removed R2: 4.7k, Resistor_SMD:R_0805_2012Metric, symbol Device:R
- added J1, J3: Conn_01x02, Connector_PinHeader_2.54mm:PinHeader_1x02_P2.54mm_Vertical, symbol Connector_Generic:Conn_01x03
- added J2: Conn_01x02, Connector_PinHeader_2.54mm:PinHeader_1x02_P2.54mm_Vertical, symbol Connector_Generic:Conn_01x02
Connections:
- net ADC_MISO: now also J3.2 (Pin_2); no longer U4.26 (34)
- net ADC_SCK: now also J1.2 (Pin_2); no longer U4.29 (37)
- net DAC_SCK: now also J1.1 (Pin_1); no longer U4.23 (31_CTX3)
- net DAC_SYNC: now also U4.30 (38); no longer U4.38 (16_A2_RX4_SCL1)
- net ADC_RANGE: now reaches U6.8 (RANGE)
- net ADC_RANGE: now also U4.29 (37)
- net DAC_SDOUT: no longer names the net of U3.16 (SDO)
- net DAC_SDOUT: no longer U4.33 (41)
- new net MISO1: J3.1 (Pin_1), U4.33 (41)
- new net MISO2: J2.1 (Pin_1), J3.3 (Pin_3)
- new net SCK2: J1.3 (Pin_3), J2.2 (Pin_2)
- no-connect marks 44 -> 47
Other:
- note added: "SPI1"
- note added: "SPI2"
- note added: "Select SPI1 for ADC to use SPI1 (share with DAC)\nSelect SPI2 for ADC to use SPI2 (share with flash mem on T4.1 underside)"
- note added: "if you are using SPI2 for ADC:\nconnect MISO2 to pin 54 \nconnect SCK2 to pin 49\n(underneath teensy 4.1)"
Changed lines of the file:
@@
 Text Label 7700 1650 2    49   ~ 0
 TFT_CS
-Text Label 7700 2750 2    49   ~ 0
-DAC_SCK
 Text Label 7700 2650 2    49   ~ 0
 DAC_SDIN
-Text Label 9900 3150 0    49   ~ 0
+Text Label 8600 4450 0    49   ~ 0
 ADC_MISO
-Text Label 9900 2850 0    49   ~ 0
-ADC_SCK
-Text Label 9900 2950 0    49   ~ 0
+Text Label 9950 2950 0    49   ~ 0
 ADC_CS
 Text Label 7700 1050 2    49   ~ 0
@@
 Text Label 7700 1550 2    49   ~ 0
 ADC_CONVST
-Text Label 9900 1950 0    49   ~ 0
+Text Label 9950 2750 0    49   ~ 0
 DAC_SYNC
-Text Label 9900 2450 0    49   ~ 0
-DAC_SDOUT
 $Comp
 L Connector_Generic:Conn_02x08_Odd_Even J28
@@
 Wire Notes Line
 	19900 2650 23850 2650
-Wire Wire Line
-	7700 3150 7450 3150
-Wire Wire Line
-	7450 3150 7450 2750
-Wire Wire Line
-	7450 2750 7700 2750
 NoConn ~ 7700 1750
 NoConn ~ 7700 1850
@@
 	1000 3350 1200 3350
 Wire Wire Line
-	550  4050 1200 4050
+	1150 4050 1200 4050
 Wire Wire Line
 	1200 4150 1200 4250
@@
 	1    0    0    -1
 $EndComp
-Text Label 4750 3500 2    50   ~ 0
-DAC_SDOUT
 NoConn ~ 4750 4300
 NoConn ~ 4750 4200
@@
 	3800 5500 3800 500
 Wire Notes Line
-	7000 4750 11200 4750
-Wire Notes Line
 	7100 5700 11300 5700
 Wire Notes Line
@@
 Wire Wire Line
 	850  3750 1200 3750
-$Comp
-L Device:R R2
-U 1 1 5F5296C2
-P 550 3150
-F 0 "R2" H 550 3000 50  0000 L CNN
-F 1 "4.7k" V 550 3050 50  0000 L CNN
-F 2 "Resistor_SMD:R_0805_2012Metric" V 480 3150 50  0001 C CNN
-F 3 "~" H 550 3150 50  0001 C CNN
-	1    550  3150
-	1    0    0    -1
-$EndComp
 $Comp
 L power:GND #PWR02
@@
 Connection ~ 850  3000
 Wire Wire Line
-	550  3300 550  4050
-Wire Wire Line
 	700  3950 1200 3950
 Wire Wire Line
 	700  3300 700  3950
 Wire Wire Line
-	550  3000 700  3000
-Wire Wire Line
 	700  3000 850  3000
-Connection ~ 700  3000
 $Comp
 L Device:R R1
@@
 ENC1SW
 NoConn ~ 9900 2650
-NoConn ~ 9900 2750
+$Comp
+L Connector_Generic:Conn_01x03 J3
+U 1 1 5F865698
+P 8400 4450
+F 0 "J3" V 8272 4262 50  0000 R CNN
+F 1 "Conn_01x02" V 8363 4262 50  0001 R CNN
+F 2 "Connector_PinHeader_2.54mm:PinHeader_1x02_P2.54mm_Vertical" H 8400 4450 50  0001 C CNN
+F 3 "~" H 8400 4450 50  0001 C CNN
+	1    8400 4450
+	-1   0    0    -1
+$EndComp
+$Comp
+L Connector_Generic:Conn_01x03 J1
+U 1 1 5F866946
+P 7700 4450
+F 0 "J1" V 7572 4262 50  0000 R CNN
+F 1 "Conn_01x02" V 7663 4262 50  0001 R CNN
+F 2 "Connector_PinHeader_2.54mm:PinHeader_1x02_P2.54mm_Vertical" H 7700 4450 50  0001 C CNN
+F 3 "~" H 7700 4450 50  0001 C CNN
+	1    7700 4450
+	-1   0    0    -1
+$EndComp
+Text Label 7950 4450 0    49   ~ 0
+ADC_SCK
+Text Label 9900 2450 0    49   ~ 0
+MISO1
+Wire Wire Line
+	7900 4350 7950 4350
+Wire Wire Line
+	7900 4550 7950 4550
+Wire Wire Line
+	8600 4350 8650 4350
+Wire Wire Line
+	8600 4550 8650 4550
+$Comp
+L Connector_Generic:Conn_01x02 J2
+U 1 1 5F88EBDB
+P 8400 3800
+F 0 "J2" V 8272 3612 50  0000 R CNN
+F 1 "Conn_01x02" V 8363 3612 50  0001 R CNN
+F 2 "Connector_PinHeader_2.54mm:PinHeader_1x02_P2.54mm_Vertical" H 8400 3800 50  0001 C CNN
+F 3 "~" H 8400 3800 50  0001 C CNN
+	1    8400 3800
+	-1   0    0    -1
+$EndComp
+Text Label 8600 3800 0    49   ~ 0
+MISO2
+Text Label 8600 3900 0    49   ~ 0
+SCK2
+Text Notes 8250 3700 0    49   ~ 0
+if you are using SPI2 for ADC:\nconnect MISO2 to pin 54 \nconnect SCK2 to pin 49\n(underneath teensy 4.1)
+Text Label 7950 4550 0    49   ~ 0
+SCK2
+Wire Wire Line
+	7900 4450 7950 4450
+Text Label 7950 4350 0    49   ~ 0
+DAC_SCK
+Text Label 8650 4550 0    49   ~ 0
+MISO2
+Text Label 8650 4350 0    49   ~ 0
+MISO1
+Text Notes 7700 4250 0    49   ~ 0
+Select SPI1 for ADC to use SPI1 (share with DAC)\nSelect SPI2 for ADC to use SPI2 (share with flash mem on T4.1 underside)
+Text Notes 7450 4400 0    49   ~ 0
+SPI1
+Text Notes 7450 4600 0    49   ~ 0
+SPI2
+Wire Wire Line
+	9900 2950 9950 2950
+Text Label 1150 4050 2    49   ~ 0
+ADC_RANGE
+Text Label 9950 2850 0    49   ~ 0
+ADC_RANGE
+Wire Wire Line
+	9900 2850 9950 2850
+Wire Notes Line
+	7000 4750 11200 4750
+NoConn ~ 4750 3500
+Text Label 7700 2750 2    49   ~ 0
+DAC_SCK
+Wire Wire Line
+	9900 2750 9950 2750
+NoConn ~ 9900 3150
+NoConn ~ 7700 3150
+NoConn ~ 9900 1950
 $EndSCHEMATC

Commit message: correct footprint to pin headers for jumpers
Parts:
- J1, J3: value Conn_01x02 -> Conn_01x03; footprint Connector_PinHeader_2.54mm:PinHeader_1x02_P2.54mm_Vertical -> Pin_Headers:Pin_Header_Straight_1x03_Pitch2.54mm
- J2: footprint Connector_PinHeader_2.54mm:PinHeader_1x02_P2.54mm_Vertical -> Pin_Headers:Pin_Header_Straight_1x02_Pitch2.54mm
Changed lines of the file:
@@
 P 8400 4450
 F 0 "J3" V 8272 4262 50  0000 R CNN
-F 1 "Conn_01x02" V 8363 4262 50  0001 R CNN
-F 2 "Connector_PinHeader_2.54mm:PinHeader_1x02_P2.54mm_Vertical" H 8400 4450 50  0001 C CNN
+F 1 "Conn_01x03" V 8363 4262 50  0001 R CNN
+F 2 "Pin_Headers:Pin_Header_Straight_1x03_Pitch2.54mm" H 8400 4450 50  0001 C CNN
 F 3 "~" H 8400 4450 50  0001 C CNN
 	1    8400 4450
@@
 P 7700 4450
 F 0 "J1" V 7572 4262 50  0000 R CNN
-F 1 "Conn_01x02" V 7663 4262 50  0001 R CNN
-F 2 "Connector_PinHeader_2.54mm:PinHeader_1x02_P2.54mm_Vertical" H 7700 4450 50  0001 C CNN
+F 1 "Conn_01x03" V 7663 4262 50  0001 R CNN
+F 2 "Pin_Headers:Pin_Header_Straight_1x03_Pitch2.54mm" H 7700 4450 50  0001 C CNN
 F 3 "~" H 7700 4450 50  0001 C CNN
 	1    7700 4450
@@
 F 0 "J2" V 8272 3612 50  0000 R CNN
 F 1 "Conn_01x02" V 8363 3612 50  0001 R CNN
-F 2 "Connector_PinHeader_2.54mm:PinHeader_1x02_P2.54mm_Vertical" H 8400 3800 50  0001 C CNN
+F 2 "Pin_Headers:Pin_Header_Straight_1x02_Pitch2.54mm" H 8400 3800 50  0001 C CNN
 F 3 "~" H 8400 3800 50  0001 C CNN
 	1    8400 3800

Commit message: rerouted pcb
Parts:
- C19, C21, C23, C25, C31, C32, C33, C34: footprint Capacitor_SMD:C_0805_2012Metric -> Capacitors_THT:CP_Radial_D5.0mm_P2.00mm
Changed lines of the file:
@@
 F 0 "C33" H 6815 4696 50  0000 L CNN
 F 1 "10u" H 6815 4605 50  0000 L CNN
-F 2 "Capacitor_SMD:C_0805_2012Metric" H 6738 4500 50  0001 C CNN
+F 2 "Capacitors_THT:CP_Radial_D5.0mm_P2.00mm" H 6738 4500 50  0001 C CNN
 F 3 "~" H 6700 4650 50  0001 C CNN
 	1    6700 4650
@@
 F 0 "C32" H 6250 4700 50  0000 L CNN
 F 1 "0.1u" H 6250 4600 50  0000 L CNN
-F 2 "Capacitor_SMD:C_0805_2012Metric" H 6538 4500 50  0001 C CNN
+F 2 "Capacitors_THT:CP_Radial_D5.0mm_P2.00mm" H 6538 4500 50  0001 C CNN
 F 3 "~" H 6500 4650 50  0001 C CNN
 	1    6500 4650
@@
 $EndComp
 $Comp
-L Device:C C20
-U 1 1 5F009DEB
-P 4200 5250
-F 0 "C20" H 3950 5300 50  0000 L CNN
-F 1 "10u" H 3950 5200 50  0000 L CNN
-F 2 "Capacitor_SMD:C_0805_2012Metric" H 4238 5100 50  0001 C CNN
-F 3 "~" H 4200 5250 50  0001 C CNN
-	1    4200 5250
-	1    0    0    -1
-$EndComp
-$Comp
 L Device:C C23
 U 1 1 5F0093E0
@@
 F 0 "C23" H 4515 4646 50  0000 L CNN
 F 1 "0.1u" H 4515 4555 50  0000 L CNN
-F 2 "Capacitor_SMD:C_0805_2012Metric" H 4438 4450 50  0001 C CNN
+F 2 "Capacitors_THT:CP_Radial_D5.0mm_P2.00mm" H 4438 4450 50  0001 C CNN
 F 3 "~" H 4400 4600 50  0001 C CNN
 	1    4400 4600
@@
 F 0 "C19" H 3900 4650 50  0000 L CNN
 F 1 "10u" H 3900 4550 50  0000 L CNN
-F 2 "Capacitor_SMD:C_0805_2012Metric" H 4238 4450 50  0001 C CNN
+F 2 "Capacitors_THT:CP_Radial_D5.0mm_P2.00mm" H 4238 4450 50  0001 C CNN
 F 3 "~" H 4200 4600 50  0001 C CNN
 	1    4200 4600
@@
 F 0 "C34" H 6815 2146 50  0000 L CNN
 F 1 "10u" H 6815 2055 50  0000 L CNN
-F 2 "Capacitor_SMD:C_0805_2012Metric" H 6738 1950 50  0001 C CNN
+F 2 "Capacitors_THT:CP_Radial_D5.0mm_P2.00mm" H 6738 1950 50  0001 C CNN
 F 3 "~" H 6700 2100 50  0001 C CNN
 	1    6700 2100
@@
 F 0 "C21" H 3900 2150 50  0000 L CNN
 F 1 "10u" H 3900 2050 50  0000 L CNN
-F 2 "Capacitor_SMD:C_0805_2012Metric" H 4188 1950 50  0001 C CNN
+F 2 "Capacitors_THT:CP_Radial_D5.0mm_P2.00mm" H 4188 1950 50  0001 C CNN
 F 3 "~" H 4150 2100 50  0001 C CNN
 	1    4150 2100
@@
 F 0 "C31" H 6250 2150 50  0000 L CNN
 F 1 "0.1u" H 6250 2050 50  0000 L CNN
-F 2 "Capacitor_SMD:C_0805_2012Metric" H 6538 1950 50  0001 C CNN
+F 2 "Capacitors_THT:CP_Radial_D5.0mm_P2.00mm" H 6538 1950 50  0001 C CNN
 F 3 "~" H 6500 2100 50  0001 C CNN
 	1    6500 2100
@@
 F 0 "C25" H 4465 2146 50  0000 L CNN
 F 1 "0.1u" H 4465 2055 50  0000 L CNN
-F 2 "Capacitor_SMD:C_0805_2012Metric" H 4388 1950 50  0001 C CNN
+F 2 "Capacitors_THT:CP_Radial_D5.0mm_P2.00mm" H 4388 1950 50  0001 C CNN
 F 3 "~" H 4350 2100 50  0001 C CNN
 	1    4350 2100
@@
 NoConn ~ 7700 3150
 NoConn ~ 9900 1950
+$Comp
+L Device:C C20
+U 1 1 5F009DEB
+P 4200 5250
+F 0 "C20" H 3950 5300 50  0000 L CNN
+F 1 "10u" H 3950 5200 50  0000 L CNN
+F 2 "Capacitor_SMD:C_0805_2012Metric" H 4238 5100 50  0001 C CNN
+F 3 "~" H 4200 5250 50  0001 C CNN
+	1    4200 5250
+	1    0    0    -1
+$EndComp
 $EndSCHEMATC

Commit message: MISO corrected from pin 41 to pin 39, teensy symbol corrections
Connections:
- net MISO1: now also U4.31 (39); no longer U4.33 (41)
Changed lines of the file:
@@
 Text Label 7700 3050 2    49   ~ 0
 ENC1SW
-NoConn ~ 9900 2650
+NoConn ~ 9900 2450
 $Comp
 L Connector_Generic:Conn_01x03 J3
@@
 Text Label 7950 4450 0    49   ~ 0
 ADC_SCK
-Text Label 9900 2450 0    49   ~ 0
+Text Label 9950 2650 0    49   ~ 0
 MISO1
 Wire Wire Line
@@
 	1    0    0    -1
 $EndComp
+Wire Wire Line
+	9900 2650 9950 2650
 $EndSCHEMATC

Commit message: schematic: change dac bypass to polarized cap and change polarity
Parts:
- C19, C21, C23, C25, C31, C32, C33, C34: symbol Device:C -> Device:CP
Connections:
- net -12V: now also C31.2, C32.2, C33.2, C34.2; no longer C31.1, C32.1, C33.1, C34.1
- net GND: now also C31.1, C32.1, C33.1, C34.1; no longer C31.2, C32.2, C33.2, C34.2
Changed lines of the file:
@@
 $EndComp
 $Comp
-L Device:C C33
+L Device:CP C33
 U 1 1 5F01A320
 P 6700 4650
-F 0 "C33" H 6815 4696 50  0000 L CNN
-F 1 "10u" H 6815 4605 50  0000 L CNN
+F 0 "C33" H 6450 4700 50  0000 L CNN
+F 1 "10u" H 6450 4600 50  0000 L CNN
 F 2 "Capacitors_THT:CP_Radial_D5.0mm_P2.00mm" H 6738 4500 50  0001 C CNN
 F 3 "~" H 6700 4650 50  0001 C CNN
 	1    6700 4650
-	1    0    0    -1
-$EndComp
-$Comp
-L Device:C C32
+	-1   0    0    1
+$EndComp
+$Comp
+L Device:CP C32
 U 1 1 5F0199E8
 P 6500 4650
-F 0 "C32" H 6250 4700 50  0000 L CNN
-F 1 "0.1u" H 6250 4600 50  0000 L CNN
+F 0 "C32" H 6600 4700 50  0000 L CNN
+F 1 "0.1u" H 6600 4600 50  0000 L CNN
 F 2 "Capacitors_THT:CP_Radial_D5.0mm_P2.00mm" H 6538 4500 50  0001 C CNN
 F 3 "~" H 6500 4650 50  0001 C CNN
 	1    6500 4650
-	1    0    0    -1
+	-1   0    0    1
 $EndComp
 $Comp
@@
 $EndComp
 $Comp
-L Device:C C23
+L Device:CP C23
 U 1 1 5F0093E0
 P 4400 4600
@@
 $EndComp
 $Comp
-L Device:C C19
+L Device:CP C19
 U 1 1 5F008568
 P 4200 4600
@@
 $EndComp
 $Comp
-L Device:C C34
+L Device:CP C34
 U 1 1 5EFF5A69
 P 6700 2100
-F 0 "C34" H 6815 2146 50  0000 L CNN
-F 1 "10u" H 6815 2055 50  0000 L CNN
+F 0 "C34" H 6450 2150 50  0000 L CNN
+F 1 "10u" H 6450 2050 50  0000 L CNN
 F 2 "Capacitors_THT:CP_Radial_D5.0mm_P2.00mm" H 6738 1950 50  0001 C CNN
 F 3 "~" H 6700 2100 50  0001 C CNN
 	1    6700 2100
-	1    0    0    -1
+	-1   0    0    1
 $EndComp
 $Comp
@@
 $EndComp
 $Comp
-L Device:C C21
+L Device:CP C21
 U 1 1 5EFF14C2
 P 4150 2100
@@
 $EndComp
 $Comp
-L Device:C C31
+L Device:CP C31
 U 1 1 5EFEC162
 P 6500 2100
-F 0 "C31" H 6250 2150 50  0000 L CNN
-F 1 "0.1u" H 6250 2050 50  0000 L CNN
+F 0 "C31" H 6600 2150 50  0000 L CNN
+F 1 "0.1u" H 6600 2050 50  0000 L CNN
 F 2 "Capacitors_THT:CP_Radial_D5.0mm_P2.00mm" H 6538 1950 50  0001 C CNN
 F 3 "~" H 6500 2100 50  0001 C CNN
 	1    6500 2100
-	1    0    0    -1
-$EndComp
-$Comp
-L Device:C C25
+	-1   0    0    1
+$EndComp
+$Comp
+L Device:CP C25
 U 1 1 5EFEB20A
 P 4350 2100
